Commit message: [CB]: Updated xacro file with measurements from wheel odom to LIDAR and IMU

File: config/robot.urdf.xacro (robot description, xacro)
@@ -2,34 +2,28 @@
 <robot name="lio" xmlns:xacro="http://tixiaoshan.github.io/">
   <xacro:property name="PI" value="3.1415926535897931" />
-  <link name="chassis_link"></link>
+  <link name="base_footprint"/>
   <link name="base_link"></link>
   <joint name="base_link_joint" type="fixed">
+    <parent link="base_footprint"/>
+    <child link="base_link" />
+    <origin xyz="0 0 0" rpy="0 0 0" />
+  </joint>
+  <link name="wheel_odom_link"/>
+  <joint name="wheel_odom_link_joint" type="fixed">
     <parent link="base_link"/>
-    <child link="chassis_link" />
-    <origin xyz="0 0 0" rpy="0 0 0" />
+    <child link="wheel_odom_link"/>
+    <origin xyz="0 0 0" rpy="0 0 0"/>
   </joint>
   <link name="lidar_link"> </link>
   <joint name="lidar_joint" type="fixed">
-    <parent link="base_link" />
+    <parent link="wheel_odom_link" />
     <child link="lidar_link" />
-    <origin xyz="0 0 0" rpy="0 0 0" />
+    <origin xyz="0.525 -0.474 1.462" rpy="0 0 0" />
   </joint>
   <link name="imu_link"> </link>
   <joint name="imu_joint" type="fixed">
-    <parent link="chassis_link" />
+    <parent link="lidar_link" />
     <child link="imu_link" />
-    <origin xyz="0 0 0" rpy="0 0 0" />
-  </joint>
-  <link name="laser_sensor_frame"> </link>
-  <joint name="laser_joint" type="fixed">
-    <parent link="imu_link" />
-    <child link="laser_sensor_frame" />
-    <origin xyz="0 0 0" rpy="0 0 0" />
-  </joint>
-  <link name="navsat_link"> </link>
-  <joint name="navsat_joint" type="fixed">
-    <parent link="chassis_link" />
-    <child link="navsat_link" />
-    <origin xyz="0 0 0" rpy="0 0 0" />
+    <origin xyz="0.0025 0 0.0929" rpy="3.141592 0 1.570769" />
   </joint>
 </robot>
